File: hw/2023/ctfBadge/version4.sch (EAGLE design)
At the start: 81 parts, among them J2 SSW-103-22-F-D-VS-K-TRCON3_SS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, J3 TYPE-C-31-M-12, Q1 mmbt2222, Q2 mmbt2222, SW2 KMR2, U1 CH340C, U10 WS2812-2020, U11 WS2812-2020, U12 WS2812-2020, U13 WS2812-2020, U14 WS2812-2020, U15 WS2812-2020, U16 WS2812-2020, U17 WS2812-2020, U18 WS2812-2020, U19 WS2812-2020, U2 AP2112-3.3, U20 WS2812-2020, U21 WS2812-2020, U22 WS2812-2020, U23 WS2812-2020, U24 WS2812-2020, U25 WS2812-2020, U26 WS2812-2020, U3 24792479PCB_37P49X52P63_KEY, U4 SMF05CT1G, U5 PCM12SMTRPCM12SMTR_CNK, U6 WS2812-2020, U7 WS2812-2020, U8 WS2812-2020, U9 WS2812-2020, X2 ESP32_WROOM32_SKINNY

Commit message: CTF-Badge modified
- 3x AAA and removed charging circuit
- USB-c
Parts:
- removed U3: 24792479PCB_37P49X52P63_KEY, 36-2479-ND_AAA-3x:24792479PCB_37P49X52P63_KEY
- added U27, U28, U29: 10201020_KEY, 36-1020-ND:10201020_KEY
Connections:
- removed net N$39: U7.DO, U9.DI
- new net N$10: U28.2, U29.1
- new net N$11: U27.2, U28.1
- new net N$9: U22.DO, U23.DI
- net GND: now also U29.2; no longer U3.2
- net N$1: now also U7.DO; no longer U22.DO
- net N$2: now also U9.DI; no longer U23.DI
- net VBAT: now also U27.1; no longer U3.1
Other:
- note added: "Digikey:"
- note added: "Digikey: 36-1020-ND"
- moved on the sheet: U10, U11, U23, U24, U25, U26, U8, U9

Commit message: gerbers generated and ready for JLCPCB
- switched 0805 parts to 0603
- gave values to neopixel capacitors
- DRC check
Parts:
- removed C25: 1uF, microbuilder:CAP_CERAMIC0805-NOOUTLINE
- removed C29: 0.1uF, microbuilder:CAP_CERAMIC0805-NOOUTLINE
- added C8: 1uF, microbuilder:CAP_CERAMIC0603_NO
- added C9: 0.1uF, rcl:C-EUC0603
- C1, C10, C11, C12, C13, C14, C15, C16, C17, C19, C2, C20, C21, C22, C23, C24, C3, C4, C5, C6, C7: value (none) -> 0.1uF
- R13, R14: value 1K -> 5.1K
Connections:
- net 3.3V: now also C9.1; no longer C29.1
- net GND: now also C8.2, C9.2; no longer C25.2, C29.2
- net VDD: now also C8.1; no longer C25.1
Other:
- note added: "Mnfr: Korean Hroparts Elec Part#: TYPE-C-31-M-12 JLCPCB#: C165948"
- note added: "todo: standard c29 to 0603"
- note removed: "Mnfr: Korean Hroparts Elec Part#: TYPE-C-31-M-14 JLCPCB#: C223907"
