File: hw/2023/ctfBadge/version4.brd (EAGLE design)
At the start: 80 x 305 mm, 81 parts, among them J2 SSW-103-22-F-D-VS-K-TRCON3_SS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, J3 TYPE-C-31-M-12, Q1 mmbt2222, Q2 mmbt2222, SW2 KMR2, U1 CH340C, U10 WS2812-2020, U11 WS2812-2020, U12 WS2812-2020, U13 WS2812-2020, U14 WS2812-2020, U15 WS2812-2020, U16 WS2812-2020, U17 WS2812-2020, U18 WS2812-2020, U19 WS2812-2020, U2 AP2112-3.3, U20 WS2812-2020, U21 WS2812-2020, U22 WS2812-2020, U23 WS2812-2020, U24 WS2812-2020, U25 WS2812-2020, U26 WS2812-2020, U3 24792479PCB_37P49X52P63_KEY, U4 SMF05CT1G, U5 PCM12SMTRPCM12SMTR_CNK, U6 WS2812-2020, U7 WS2812-2020, U8 WS2812-2020, U9 WS2812-2020, X2 ESP32_WROOM32_SKINNY

Commit message: Added test firmware
Parts:
- moved R2 171.3 mm to (0.00, -180.3)
- moved R4 171.3 mm to (0.00, -182.9)
- moved J3 140.8 mm to (-5.08, -203.2)
- moved D2 22.9 mm to (15.2, -48.3)
- moved D6 20.5 mm to (12.1, -45.1)
Changed lines of the file:
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@@
 <attribute name="VALUE" x="-2.17548125" y="-286.958090625" size="1.27075" layer="27"/>
 </element>
-<element name="D2" library="microbuilder" package="SOD-123" value="MBR120" x="38.1" y="-48.26" smashed="yes">
-<attribute name="NAME" x="36.83" y="-47.244" size="0.8128" layer="25" ratio="18"/>
-<attribute name="VALUE" x="36.83" y="-50.038" size="0.4064" layer="27" ratio="10"/>
+<element name="D2" library="microbuilder" package="SOD-123" value="MBR120" x="15.24" y="-48.26" smashed="yes">
+<attribute name="NAME" x="13.97" y="-47.244" size="0.8128" layer="25" ratio="18"/>
+<attribute name="VALUE" x="13.97" y="-50.038" size="0.4064" layer="27" ratio="10"/>
 </element>
 <element name="U3" library="36-2479-ND_AAA-3x" package="2479PCB_37P49X52P63_KEY" value="24792479PCB_37P49X52P63_KEY" x="12.7" y="-218.44" smashed="yes" rot="R180">
@@
 <attribute name="VALUE" x="15.3813" y="-220.98" size="1.27" layer="21" ratio="6" rot="R180"/>
 </element>
-<element name="D6" library="microbuilder" package="SOD-123" value="MBR120" x="32.385" y="-47.625" smashed="yes">
-<attribute name="NAME" x="31.115" y="-46.609" size="0.8128" layer="25" ratio="18"/>
-<attribute name="VALUE" x="31.115" y="-49.403" size="0.4064" layer="27" ratio="10"/>
+<element name="D6" library="microbuilder" package="SOD-123" value="MBR120" x="12.065" y="-45.085" smashed="yes">
+<attribute name="NAME" x="10.795" y="-44.069" size="0.8128" layer="25" ratio="18"/>
+<attribute name="VALUE" x="10.795" y="-46.863" size="0.4064" layer="27" ratio="10"/>
 </element>
-<element name="J3" library="TYPE-C-31-M-12" package="HRO_TYPE-C-31-M-12" value="TYPE-C-31-M-12" x="-93.98" y="-312.42" smashed="yes">
-<attribute name="MANUFACTURER" value="HRO Electronics Co., Ltd." x="-93.98" y="-312.42" size="1.778" layer="27" display="off"/>
-<attribute name="MAXIMUM_PACKAGE_HEIGHT" value="3.26 mm" x="-93.98" y="-312.42" size="1.778" layer="27" display="off"/>
-<attribute name="NAME" x="-99.005" y="-305.85" size="1.27" layer="25"/>
-<attribute name="PARTREV" value="2020.12.08" x="-93.98" y="-312.42" size="1.778" layer="27" display="off"/>
-<attribute name="SNAPEDA_PN" value="TYPE-C-31-M-12" x="-93.98" y="-312.42" size="1.778" layer="27" display="off"/>
-<attribute name="STANDARD" value="Manufacturer Recommendations" x="-93.98" y="-312.42" size="1.778" layer="27" display="off"/>
-<attribute name="VALUE" x="-99.005" y="-315.47" size="1.27" layer="27" align="top-left"/>
+<element name="J3" library="TYPE-C-31-M-12" package="HRO_TYPE-C-31-M-12" value="TYPE-C-31-M-12" x="-5.08" y="-203.2" smashed="yes">
+<attribute name="MANUFACTURER" value="HRO Electronics Co., Ltd." x="-5.08" y="-203.2" size="1.778" layer="27" display="off"/>
+<attribute name="MAXIMUM_PACKAGE_HEIGHT" value="3.26 mm" x="-5.08" y="-203.2" size="1.778" layer="27" display="off"/>
+<attribute name="NAME" x="-10.105" y="-196.63" size="1.27" layer="25"/>
+<attribute name="PARTREV" value="2020.12.08" x="-5.08" y="-203.2" size="1.778" layer="27" display="off"/>
+<attribute name="SNAPEDA_PN" value="TYPE-C-31-M-12" x="-5.08" y="-203.2" size="1.778" layer="27" display="off"/>
+<attribute name="STANDARD" value="Manufacturer Recommendations" x="-5.08" y="-203.2" size="1.778" layer="27" display="off"/>
+<attribute name="VALUE" x="-10.105" y="-206.25" size="1.27" layer="27" align="top-left"/>
 </element>
-<element name="R2" library="microbuilder" package="0603-NO" value="5.1K" x="-99.06" y="-320.04" smashed="yes">
-<attribute name="NAME" x="-97.282" y="-320.167" size="0.8128" layer="25" font="vector" ratio="18"/>
-<attribute name="VALUE" x="-97.282" y="-320.802" size="0.4064" layer="27" font="vector" ratio="10"/>
+<element name="R2" library="microbuilder" package="0603-NO" value="5.1K" x="0" y="-180.34" smashed="yes">
+<attribute name="NAME" x="1.778" y="-180.467" size="0.8128" layer="25" font="vector" ratio="18"/>
+<attribute name="VALUE" x="1.778" y="-181.102" size="0.4064" layer="27" font="vector" ratio="10"/>
 </element>
-<element name="R4" library="microbuilder" package="0603-NO" value="5.1K" x="-99.06" y="-322.58" smashed="yes">
-<attribute name="NAME" x="-97.282" y="-322.707" size="0.8128" layer="25" font="vector" ratio="18"/>
-<attribute name="VALUE" x="-97.282" y="-323.342" size="0.4064" layer="27" font="vector" ratio="10"/>
+<element name="R4" library="microbuilder" package="0603-NO" value="5.1K" x="0" y="-182.88" smashed="yes">
+<attribute name="NAME" x="1.778" y="-183.007" size="0.8128" layer="25" font="vector" ratio="18"/>
+<attribute name="VALUE" x="1.778" y="-183.642" size="0.4064" layer="27" font="vector" ratio="10"/>
 </element>
 </elements>
@@
 <wire x1="-0.915" y1="-285.03" x2="-17" y2="-256.54" width="0" layer="19" extent="1-1"/>
 <wire x1="2" y1="-288.07" x2="-0.915" y2="-285.03" width="0" layer="19" extent="1-1"/>
-<wire x1="-89.655" y1="-308.25" x2="-28.855" y2="-257.09" width="0" layer="19" extent="1-1"/>
-<wire x1="-90.78" y1="-307.67" x2="-89.655" y2="-308.25" width="0" layer="19" extent="1-1"/>
-<wire x1="-89.655" y1="-312.42" x2="-89.655" y2="-308.25" width="0" layer="19" extent="1-1"/>
-<wire x1="-97.18" y1="-307.67" x2="-90.78" y2="-307.67" width="0" layer="19" extent="1-1"/>
-<wire x1="-98.305" y1="-308.25" x2="-97.18" y2="-307.67" width="0" layer="19" extent="1-1"/>
-<wire x1="-98.305" y1="-312.42" x2="-98.305" y2="-308.25" width="0" layer="19" extent="1-1"/>
-<wire x1="-98.21" y1="-320.04" x2="-98.305" y2="-312.42" width="0" layer="19" extent="1-1"/>
-<wire x1="-98.21" y1="-322.58" x2="-98.21" y2="-320.04" width="0" layer="19" extent="1-1"/>
+<wire x1="-0.755" y1="-199.03" x2="-28.855" y2="-257.09" width="0" layer="19" extent="1-1"/>
+<wire x1="-1.88" y1="-198.45" x2="-0.755" y2="-199.03" width="0" layer="19" extent="1-1"/>
+<wire x1="-0.755" y1="-203.2" x2="-0.755" y2="-199.03" width="0" layer="19" extent="1-1"/>
+<wire x1="-8.28" y1="-198.45" x2="-1.88" y2="-198.45" width="0" layer="19" extent="1-1"/>
+<wire x1="-9.405" y1="-199.03" x2="-8.28" y2="-198.45" width="0" layer="19" extent="1-1"/>
+<wire x1="-9.405" y1="-203.2" x2="-9.405" y2="-199.03" width="0" layer="19" extent="1-1"/>
+<wire x1="0.85" y1="-180.34" x2="-9.405" y2="-203.2" width="0" layer="19" extent="1-1"/>
+<wire x1="0.85" y1="-182.88" x2="0.85" y2="-180.34" width="0" layer="19" extent="1-1"/>
 </signal>
 <signal name="VDD">
@@
 <contactref element="J3" pad="B4/A9"/>
 <contactref element="J3" pad="A4/B9"/>
-<wire x1="-91.58" y1="-307.67" x2="-96.38" y2="-307.67" width="0" layer="19" extent="1-1"/>
-<wire x1="34.235" y1="-47.625" x2="-91.58" y2="-307.67" width="0" layer="19" extent="1-1"/>
-<wire x1="16.21" y1="-29.83" x2="34.235" y2="-47.625" width="0" layer="19" extent="1-1"/>
+<wire x1="-2.68" y1="-198.45" x2="-7.48" y2="-198.45" width="0" layer="19" extent="1-1"/>
+<wire x1="13.915" y1="-45.085" x2="-2.68" y2="-198.45" width="0" layer="19" extent="1-1"/>
+<wire x1="16.21" y1="-29.83" x2="13.915" y2="-45.085" width="0" layer="19" extent="1-1"/>
 </signal>
 <signal name="VBAT">
@@
 <contactref element="U3" pad="1"/>
 <contactref element="D2" pad="A"/>
-<wire x1="39.95" y1="-48.26" x2="12.7" y2="-218.44" width="0" layer="19" extent="1-1"/>
-<wire x1="-30.195" y1="-238.125" x2="39.95" y2="-48.26" width="0" layer="19" extent="1-16"/>
+<wire x1="17.09" y1="-48.26" x2="12.7" y2="-218.44" width="0" layer="19" extent="1-1"/>
+<wire x1="-30.195" y1="-238.125" x2="17.09" y2="-48.26" width="0" layer="19" extent="1-16"/>
 </signal>
 <signal name="3.3V">
@@
 <contactref element="J3" pad="B6"/>
 <contactref element="J3" pad="A6"/>
-<wire x1="-93.23" y1="-307.67" x2="-94.23" y2="-307.67" width="0" layer="19" extent="1-1"/>
-<wire x1="-20.955" y1="-33.02" x2="-93.23" y2="-307.67" width="0" layer="19" extent="1-1"/>
+<wire x1="-4.33" y1="-198.45" x2="-5.33" y2="-198.45" width="0" layer="19" extent="1-1"/>
+<wire x1="-20.955" y1="-33.02" x2="-4.33" y2="-198.45" width="0" layer="19" extent="1-1"/>
 </signal>
 <signal name="N$29">
@@
 <contactref element="J3" pad="B7"/>
 <contactref element="J3" pad="A7"/>
-<wire x1="-93.73" y1="-307.67" x2="-94.73" y2="-307.67" width="0" layer="19" extent="1-1"/>
-<wire x1="-20.955" y1="-32.385" x2="-93.73" y2="-307.67" width="0" layer="19" extent="1-1"/>
+<wire x1="-4.83" y1="-198.45" x2="-5.83" y2="-198.45" width="0" layer="19" extent="1-1"/>
+<wire x1="-20.955" y1="-32.385" x2="-4.83" y2="-198.45" width="0" layer="19" extent="1-1"/>
 </signal>
 <signal name="RTS">
@@
 <contactref element="U5" pad="2"/>
 <contactref element="D6" pad="C"/>
-<wire x1="36.25" y1="-48.26" x2="30.535" y2="-47.625" width="0" layer="19" extent="1-1"/>
-<wire x1="-21.102734375" y1="-57.054096875" x2="36.25" y2="-48.26" width="0" layer="19" extent="1-16"/>
+<wire x1="13.39" y1="-48.26" x2="10.215" y2="-45.085" width="0" layer="19" extent="1-1"/>
+<wire x1="-21.102734375" y1="-57.054096875" x2="13.39" y2="-48.26" width="0" layer="19" extent="1-16"/>
 </signal>
 <signal name="N$6">
 <contactref element="J3" pad="B5"/>
 <contactref element="R4" pad="1"/>
-<wire x1="-92.23" y1="-307.67" x2="-99.91" y2="-322.58" width="0" layer="19" extent="1-1"/>
+<wire x1="-3.33" y1="-198.45" x2="-0.85" y2="-182.88" width="0" layer="19" extent="1-1"/>
 </signal>
 <signal name="N$8">
 <contactref element="J3" pad="A5"/>
 <contactref element="R2" pad="1"/>
-<wire x1="-95.23" y1="-307.67" x2="-99.91" y2="-320.04" width="0" layer="19" extent="1-1"/>
+<wire x1="-6.33" y1="-198.45" x2="-0.85" y2="-180.34" width="0" layer="19" extent="1-1"/>
 </signal>
 </signals>

Commit message: CTF-Badge modified
- 3x AAA and removed charging circuit
- USB-c
Parts:
- removed U3: 24792479PCB_37P49X52P63_KEY, 36-2479-ND_AAA-3x:2479PCB_37P49X52P63_KEY
- added U27, U28, U29: 10201020_KEY, 36-1020-ND:1020_KEY
- moved J3 171.8 mm to (-23.5, -32.4), turned to 284 degrees
- moved R4 150.5 mm to (-13.3, -33.0)
- moved R2 146.0 mm to (-13.3, -34.9)
- moved D2 37.1 mm to (-14.0, -25.4), turned to 270 degrees
- moved D6 34.7 mm to (-16.5, -25.4), turned to 270 degrees
- moved U6 4.33 mm to (-18.0, -70.0), turned to 180 degrees
- moved U7 2.58 mm to (18.0, -70.0), turned to 180 degrees
- moved U26 2.52 mm to (0.00, -287.0), turned to 180 degrees
- moved U13 2.51 mm to (24.0, -130.0), turned to 180 degrees
- moved C1 2.50 mm to (-29.0, -230.0)
- moved U12 2.37 mm to (-24.0, -130.0), turned to 180 degrees
- moved C7 2.24 mm to (-14.0, -70.0)
- moved C11 2.05 mm to (-23.0, -256.0)
- moved C5 2.00 mm to (14.0, -70.0)
- moved U10 1.96 mm to (-22.0, -110.0), turned to 180 degrees
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Connections:
- removed net N$39: U7.1, U9.3
- new net N$10: U28.2, U29.1
- new net N$11: U27.2, U28.1
- new net N$9: U22.1, U23.3
- net GND: now also U29.2; no longer U3.2
- net N$1: now also U7.1; no longer U22.1
- net N$2: now also U9.3; no longer U23.3
- net VBAT: now also U27.1; no longer U3.1
Routing:
- net N$3: track 0.00 -> 87.7 mm
- net N$52: track 0.00 -> 84.2 mm
- net N$50: track 0.00 -> 81.7 mm
- net N$48: track 0.00 -> 77.8 mm
- net N$46: track 0.00 -> 73.7 mm
- net N$9: track 0.00 -> 70.6 mm
- net N$44: track 0.00 -> 69.7 mm
- net N$51: track 0.00 -> 66.6 mm
- net N$42: track 0.00 -> 65.7 mm
- net N$49: track 0.00 -> 62.6 mm
- net N$40: track 0.00 -> 61.7 mm
- net N$47: track 0.00 -> 58.6 mm
- net N$4: track 0.00 -> 58.6 mm
- net N$5: track 0.00 -> 58.1 mm
- net N$1: track 0.00 -> 57.7 mm
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Other:
- board text added: "+"
- board text added: "3x AAA Input: 4.5V"
- board text added: "NORTHSEC 2022 V4"
- board text removed: "NorthSec2022"

Commit message: gerbers generated and ready for JLCPCB
- switched 0805 parts to 0603
- gave values to neopixel capacitors
- DRC check
Parts:
- removed C25: 1uF, microbuilder:0805-NO
- removed C29: 0.1uF, microbuilder:0805-NO
- added C8: 1uF, microbuilder:0603-NO
- added C9: 0.1uF, rcl:C0603
- C1, C10, C11, C12, C13, C14, C15, C16, C17, C19, C2, C20, C21, C22, C23, C24, C3, C4, C5, C6, C7: value (none) -> 0.1uF
- R13, R14: value 1K -> 5.1K
Connections:
- net 3.3V: now also C9.1; no longer C29.1
- net GND: now also C8.2, C9.2; no longer C25.2, C29.2
- net VDD: now also C8.1; no longer C25.1
Other:
- board text added: "NORTHSEC 2023 V4"
- board text removed: "NORTHSEC 2022 V4"

Commit message: generated proposed factory gerber for Rizome (silkscreen still missing)
Other:
- board text added: "NORTHSEC2023"
- board text removed: "NORTHSEC 2023 V4"
