File: hw/2023/confBadge/confBadgeV1.brd (EAGLE design)
At the start: 96.5 x 78.7 mm, 94 parts, among them J1 SSW-103-22-F-D-VS-K-TRCON3_SS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, J2 SSW-103-22-F-D-VS-K-TRCON3_SS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, J3 TYPE-C-31-M-12, Q1 8/16/20MHz, U1 ATMEGA328, U10 WS2812-2020, U11 WS2812-2020, U12 WS2812-2020, U13 WS2812-2020, U14 WS2812-2020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

Commit message: Updated design from artists
Still missing fill on Conf-badge top silkscreen
waiting on bottom silkcreen
Parts:
- moved C20 3.83 mm to (67.9, 8.26), turned to 0 degrees
- moved R19 2.54 mm to (71.8, 14.0)
- moved S3 2.54 mm to (73.7, 10.2)
- moved S4 1.27 mm to (14.0, 22.9)
- moved S5 1.27 mm to (14.0, 5.08)
- moved S6 1.27 mm to (5.08, 14.0)
- moved S7 1.27 mm to (22.9, 14.0)
Routing:
- net GND: track 114.4 -> 117.0 mm
- net BTN_A: track 39.6 -> 37.0 mm
- net BTN_D: track 54.9 -> 56.7 mm
- net RESET: track 58.8 -> 60.6 mm
- net BTN_L: track 46.7 -> 48.1 mm
- net BTN_R: track 50.4 -> 51.7 mm
- net BTN_U: track 37.7 -> 38.3 mm
Other:
- board text removed: "2023"
- board text removed: "C:/Users/lambert/Documents/GitHub/nsec-badge-dev/hw/2023/design/BadgeConf2023-01B_filled.bmp"
- board text removed: "NSEC"
- board text removed: "pssst, go to the soldering village to add your OLED screen"
